File: Placa_PIC18F4550/Placa_PIC18F4550/Placa_PIC18F4550.sch (KiCad schematic (older format))
At the start: 32 parts, among them J1 PORTD, J10 USB_B, J11 PICKIT, J2 PORTA, J3 PORTE, J4 PORTB, J5 PORTC, J6 GND, J7 Vol, J8 Volt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

Commit message: Actualicación de documentos
Changed lines of the file:
@@
 F 3 "~" H 3700 1950 50  0001 C CNN
 	1    3700 1950
-	0    1    1    0
-$EndComp
-Wire Wire Line
-	3550 1950 3450 1950
+	0    -1   -1   0
+$EndComp
 $Comp
 L power:GND #PWR0103
@@
 $EndComp
 Wire Wire Line
-	4000 1950 3850 1950
-Wire Wire Line
 	8300 4850 8100 4850
 Wire Wire Line
@@
 Text Label 10200 4800 2    50   ~ 0
 RB5
+Wire Wire Line
+	3550 1950 3450 1950
+Wire Wire Line
+	3850 1950 4000 1950
 $EndSCHEMATC

Commit message: Programa SPI
Parts:
- added J12: Conn_01x02_Male, Connector_PinHeader_2.54mm:PinHeader_1x02_P2.54mm_Vertical, symbol Connector:Conn_01x02_Male
- Q1: footprint Package_TO_SOT_THT:TO-92_Inline -> Package_TO_SOT_THT:TO-92L_Inline_Wide
Connections:
- wire segments 149 -> 150
Changed lines of the file:
@@
 F 0 "Q1" H 9941 2346 50  0000 L CNN
 F 1 "2N3906" H 9941 2255 50  0000 L CNN
-F 2 "Package_TO_SOT_THT:TO-92_Inline" H 9950 2225 50  0001 L CIN
+F 2 "Package_TO_SOT_THT:TO-92L_Inline_Wide" H 9950 2225 50  0001 L CIN
 F 3 "https://www.fairchildsemi.com/datasheets/2N/2N3906.pdf" H 9750 2300 50  0001 L CNN
 	1    9750 2300
@@
 Wire Wire Line
 	5850 5400 5850 5300
-Wire Wire Line
-	5850 4850 5850 5000
-Text Label 5850 4850 3    50   ~ 0
+Text Label 5850 4450 3    50   ~ 0
 RD0
 $Comp
@@
 Wire Wire Line
 	3850 1950 4000 1950
+$Comp
+L Connector:Conn_01x02_Male J12
+U 1 1 5CB309E6
+P 6050 4750
+F 0 "J12" H 6023 4630 50  0000 R CNN
+F 1 "Conn_01x02_Male" H 6023 4721 50  0000 R CNN
+F 2 "Connector_PinHeader_2.54mm:PinHeader_1x02_P2.54mm_Vertical" H 6050 4750 50  0001 C CNN
+F 3 "~" H 6050 4750 50  0001 C CNN
+	1    6050 4750
+	-1   0    0    1
+$EndComp
+Wire Wire Line
+	5850 4750 5850 5000
+Wire Wire Line
+	5850 4450 5850 4650
 $EndSCHEMATC
